File: Hardware/VL6180/VL6180.sch (EAGLE design)
At the start: 28 parts, among them T1 2N7002BKS, T2 2N7002BKS, U1 VL6180X, U2 VL6180X, U3 MIC5225_2.8V

Commit message: update 02-10-2017
Parts:
- removed R4: 47K, microbuilder:RESISTOR0805_NOOUTLINE
- removed TP6: GPIO1-0, SparkFun-Connectors:TEST-POINT3X4
- added C7: 470pF, resistor:C-EUC0603
- added R1: 47K, resistor:R-EU_R0603
- added U$3: 2X5, headers(2mm)(samtec):2X5
- C1: value 0.1uF -> 1uF; device microbuilder:CAP_CERAMIC0805-NOOUTLINE -> resistor:C-EUC0603
- C2: value 0.1uF -> 10uF; device microbuilder:CAP_CERAMIC0805-NOOUTLINE -> resistor:C-EUC0603
- C3: value 10uF -> 100nF; device microbuilder:CAP_CERAMIC0805-NOOUTLINE -> resistor:C-EUC0603
- C4: value 10uF -> 4.7uF; device microbuilder:CAP_CERAMIC0805-NOOUTLINE -> resistor:C-EUC0603
- C5: value 4.7uF -> 100nF; device rcl:C-EUC0603 -> resistor:C-EUC0603
- C6: device rcl:C-EUC0603 -> resistor:C-EUC0603
- H1: value 1X6 -> 1X3; device header:1X6 -> headers(.1in):1X3
- R2: device microbuilder:RESISTOR0805_NOOUTLINE -> resistor:R-EU_R0603
- T1, T2: value 2N7002BKS -> 2N7002DW
- TP1: value SDA -> SCL
- TP2: value SCL -> SDA
- TP5: value GPIO1-1 -> GND
- U3: value MIC5225_2.8V -> MIC5219_2.8V
Connections:
- new net N$2: C7.1, U3.P4
- new net SW1: H1.1, U$3.7
- new net SW2: H1.2, U$3.8
- net 2.8V: now also C2.1, C4.1, R1.2; no longer C1.2, C2.2, R4.2
- net 3.3V: now also C1.1, U$3.1, U$3.2; no longer C4.1, H1.1
- net CS0: now also U$3.5; no longer H1.4
- net CS1: now also U$3.6; no longer H1.5
- net GND: now also C1.2, C2.2, C7.2, H1.3, TP5.1, U$3.10, U$3.9; no longer C1.1, C2.1, H1.6
- net N$1: now also R1.1; no longer R2.1, TP6.1
- net N$3: now also R2.1; no longer R4.1, TP5.1
- net SCL: now also U$3.4; no longer H1.3
- net SDA: now also U$3.3; no longer H1.2
Other:
- moved on the sheet: C1, C2, C3, C4, C5, C6, R2, TP5
