File: Hardware/SWITCH/switch.sch (EAGLE design)
At the start: 4 parts, among them SW1 SWITCH-2SMD-12MM, SW2 SWITCH-2SMD-12MM

Commit message: update 02-10-2017
Parts:
- removed J1: (no value), SparkFun-Connectors:CONN_031X03_SMD_RA_MALE_POST_SMALLER
- removed JP1: JUMPER-SMT_2_NO_SILK_ROUND, SparkFun-Jumpers:JUMPER-SMT_2_NO_SILK_ROUND
- removed SW1, SW2: SWITCH-2SMD-12MM, SparkFun-Electromechanical:SWITCH-MOMENTARY-2SMD-12MM
- added H1: 1X3, headers(.1in):1X3
- added S1, S2: (no value), switch-omron:40-XX
Connections:
- removed net N$1: JP1.2, SW1.1, SW2.2
- net GND: now also H1.3, S1.S, S1.S1, S2.P, S2.P1; no longer J1.3, JP1.1
- net SW1: now also H1.1, S1.P, S1.P1; no longer J1.1, SW1.2
- net SW2: now also H1.2, S2.S, S2.S1; no longer J1.2, SW2.1
Other:
- note added: "Chaves Posição Mão"
- note added: "Conector"
- note added: "Pos. Inferior"
- note added: "Pos. Superior"
Changed lines of the file:
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@@
 <parts>
 <part name="FRAME1" library="SparkFun-Aesthetics" deviceset="FRAME-A4L" device=""/>
-<part name="SW2" library="SparkFun-Electromechanical" deviceset="SWITCH-MOMENTARY-2" device="SMD-12MM" value="SWITCH-2SMD-12MM"/>
-<part name="SW1" library="SparkFun-Electromechanical" deviceset="SWITCH-MOMENTARY-2" device="SMD-12MM" value="SWITCH-2SMD-12MM"/>
-<part name="JP1" library="SparkFun-Jumpers" deviceset="JUMPER-SMT_2_NO" device="_SILK_ROUND" value=""/>
 <part name="GND1" library="SparkFun-PowerSymbols" deviceset="GND" device=""/>
-<part name="J1" library="SparkFun-Connectors" deviceset="CONN_03" device="1X03_SMD_RA_MALE_POST_SMALLER"/>
 <part name="GND2" library="SparkFun-PowerSymbols" deviceset="GND" device=""/>
+<part name="S2" library="switch-omron" library_urn="urn:adsk.eagle:library:377" deviceset="40-XX" device=""/>
+<part name="S1" library="switch-omron" library_urn="urn:adsk.eagle:library:377" deviceset="40-XX" device=""/>
+<part name="H1" library="headers(.1in)" deviceset="1X3" device=""/>
 </parts>
 <sheets>
 <sheet>
 <plain>
+<text x="66.04" y="160.02" size="6.4516" layer="97">Chaves Posição Mão</text>
+<wire x1="-22.86" y1="81.28" x2="53.34" y2="81.28" width="0.254" layer="97" style="shortdash"/>
+<wire x1="53.34" y1="81.28" x2="233.68" y2="81.28" width="0.254" layer="97" style="shortdash"/>
+<wire x1="233.68" y1="81.28" x2="233.68" y2="152.4" width="0.254" layer="97" style="shortdash"/>
+<wire x1="233.68" y1="152.4" x2="50.8" y2="152.4" width="0.254" layer="97" style="shortdash"/>
+<wire x1="50.8" y1="152.4" x2="-22.86" y2="152.4" width="0.254" layer="97" style="shortdash"/>
+<wire x1="-22.86" y1="152.4" x2="-22.86" y2="81.28" width="0.254" layer="97" style="shortdash"/>
+<wire x1="50.8" y1="152.4" x2="53.34" y2="152.4" width="0.1524" layer="97"/>
+<wire x1="53.34" y1="152.4" x2="53.34" y2="81.28" width="0.254" layer="97" style="shortdash"/>
+<text x="0" y="147.32" size="2.1844" layer="97">Conector</text>
+<text x="111.76" y="104.14" size="1.778" layer="97">Pos. Inferior</text>
+<text x="172.72" y="104.14" size="1.778" layer="97">Pos. Superior</text>
 </plain>
 <instances>
 <instance part="FRAME1" gate="G$1" x="-27.94" y="-7.62"/>
-<instance part="SW2" gate="G$1" x="60.96" y="121.92" smashed="yes">
-<attribute name="NAME" x="58.42" y="124.46" size="1.778" layer="95"/>
-<attribute name="VALUE" x="53.34" y="114.3" size="1.778" layer="96"/>
-</instance>
-<instance part="SW1" gate="G$1" x="121.92" y="121.92" smashed="yes">
-<attribute name="NAME" x="119.38" y="124.46" size="1.778" layer="95"/>
-<attribute name="VALUE" x="114.3" y="114.3" size="1.778" layer="96"/>
-</instance>
-<instance part="JP1" gate="G$1" x="91.44" y="109.22" smashed="yes" rot="R90">
-<attribute name="NAME" x="93.98" y="111.76" size="1.778" layer="95" font="vector"/>
-<attribute name="VALUE" x="96.52" y="109.22" size="1.778" layer="96" font="vector" align="top-left"/>
-</instance>
-<instance part="GND1" gate="1" x="91.44" y="78.74"/>
-<instance part="J1" gate="J$1" x="5.08" y="45.72" rot="MR180"/>
-<instance part="GND2" gate="1" x="38.1" y="33.02"/>
+<instance part="GND1" gate="1" x="147.32" y="101.6"/>
+<instance part="GND2" gate="1" x="10.16" y="116.84"/>
+<instance part="S2" gate="1" x="116.84" y="114.3" rot="MR270"/>
+<instance part="S1" gate="1" x="177.8" y="114.3" rot="MR270"/>
+<instance part="H1" gate="G$1" x="0" y="127"/>
 </instances>
 <busses>
 </busses>
 <nets>
-<net name="N$1" class="0">
-<segment>
-<pinref part="SW2" gate="G$1" pin="2"/>
-<pinref part="SW1" gate="G$1" pin="1"/>
-<wire x1="66.04" y1="121.92" x2="91.44" y2="121.92" width="0.1524" layer="91"/>
-<wire x1="91.44" y1="121.92" x2="116.84" y2="121.92" width="0.1524" layer="91"/>
-<wire x1="91.44" y1="121.92" x2="91.44" y2="114.3" width="0.1524" layer="91"/>
-<junction x="91.44" y="121.92"/>
-<pinref part="JP1" gate="G$1" pin="2"/>
-</segment>
-</net>
 <net name="SW2" class="0">
 <segment>
-<pinref part="SW2" gate="G$1" pin="1"/>
-<wire x1="55.88" y1="121.92" x2="27.94" y2="121.92" width="0.1524" layer="91"/>
-<label x="27.94" y="121.92" size="1.778" layer="95"/>
+<label x="83.82" y="111.76" size="1.778" layer="95"/>
+<wire x1="106.68" y1="111.76" x2="104.14" y2="111.76" width="0.1524" layer="91"/>
+<wire x1="104.14" y1="111.76" x2="83.82" y2="111.76" width="0.1524" layer="91"/>
+<pinref part="S2" gate="1" pin="S1"/>
+<wire x1="111.76" y1="111.76" x2="109.22" y2="111.76" width="0.1524" layer="91"/>
+<pinref part="S2" gate="1" pin="S"/>
+<wire x1="109.22" y1="111.76" x2="106.68" y2="111.76" width="0.1524" layer="91"/>
+<wire x1="111.76" y1="114.3" x2="109.22" y2="114.3" width="0.1524" layer="91"/>
+<wire x1="109.22" y1="114.3" x2="109.22" y2="111.76" width="0.1524" layer="91"/>
+<junction x="109.22" y="111.76"/>
 </segment>
 <segment>
-<pinref part="J1" gate="J$1" pin="2"/>
-<wire x1="12.7" y1="45.72" x2="33.02" y2="45.72" width="0.1524" layer="91"/>
-<label x="27.94" y="45.72" size="1.778" layer="95"/>
+<wire x1="2.54" y1="127" x2="22.86" y2="127" width="0.1524" layer="91"/>
+<label x="17.78" y="127" size="1.778" layer="95"/>
+<pinref part="H1" gate="G$1" pin="2"/>
 </segment>
 </net>
 <net name="SW1" class="0">
 <segment>
-<pinref part="SW1" gate="G$1" pin="2"/>
-<wire x1="127" y1="121.92" x2="142.24" y2="121.92" width="0.1524" layer="91"/>
-<wire x1="142.24" y1="121.92" x2="142.24" y2="149.86" width="0.1524" layer="91"/>
-<wire x1="142.24" y1="149.86" x2="27.94" y2="149.86" width="0.1524" layer="91"/>
-<label x="27.94" y="149.86" size="1.778" layer="95"/>
+<wire x1="187.96" y1="111.76" x2="198.12" y2="111.76" width="0.1524" layer="91"/>
+<wire x1="198.12" y1="111.76" x2="198.12" y2="121.92" width="0.1524" layer="91"/>
+<wire x1="198.12" y1="121.92" x2="198.12" y2="124.46" width="0.1524" layer="91"/>
+<wire x1="198.12" y1="124.46" x2="198.12" y2="139.7" width="0.1524" layer="91"/>
+<wire x1="198.12" y1="139.7" x2="83.82" y2="139.7" width="0.1524" layer="91"/>
+<label x="83.82" y="139.7" size="1.778" layer="95"/>
+<pinref part="S1" gate="1" pin="P1"/>
+<wire x1="182.88" y1="111.76" x2="185.42" y2="111.76" width="0.1524" layer="91"/>
+<pinref part="S1" gate="1" pin="P"/>
+<wire x1="185.42" y1="111.76" x2="187.96" y2="111.76" width="0.1524" layer="91"/>
+<wire x1="182.88" y1="114.3" x2="185.42" y2="114.3" width="0.1524" layer="91"/>
+<wire x1="185.42" y1="114.3" x2="185.42" y2="111.76" width="0.1524" layer="91"/>
+<junction x="185.42" y="111.76"/>
 </segment>
 <segment>
-<pinref part="J1" gate="J$1" pin="1"/>
-<wire x1="12.7" y1="48.26" x2="33.02" y2="48.26" width="0.1524" layer="91"/>
-<label x="27.94" y="48.26" size="1.778" layer="95"/>
+<wire x1="2.54" y1="129.54" x2="22.86" y2="129.54" width="0.1524" layer="91"/>
+<label x="17.78" y="129.54" size="1.778" layer="95"/>
+<pinref part="H1" gate="G$1" pin="1"/>
 </segment>
 </net>
 <net name="GND" class="0">
 <segment>
-<wire x1="88.9" y1="88.9" x2="27.94" y2="88.9" width="0.1524" layer="91"/>
-<label x="27.94" y="88.9" size="1.778" layer="95"/>
-<pinref part="JP1" gate="G$1" pin="1"/>
-<wire x1="91.44" y1="104.14" x2="91.44" y2="88.9" width="0.1524" layer="91"/>
-<wire x1="91.44" y1="88.9" x2="88.9" y2="88.9" width="0.1524" layer="91"/>
-<pinref part="GND1" gate="1" pin="GND"/>
-<wire x1="91.44" y1="81.28" x2="91.44" y2="88.9" width="0.1524" layer="91"/>
-<junction x="91.44" y="88.9"/>
+<pinref part="GND2" gate="1" pin="GND"/>
+<wire x1="2.54" y1="124.46" x2="10.16" y2="124.46" width="0.1524" layer="91"/>
+<wire x1="10.16" y1="124.46" x2="10.16" y2="119.38" width="0.1524" layer="91"/>
+<pinref part="H1" gate="G$1" pin="3"/>
 </segment>
 <segment>
-<pinref part="J1" gate="J$1" pin="3"/>
-<wire x1="12.7" y1="43.18" x2="33.02" y2="43.18" width="0.1524" layer="91"/>
-<label x="27.94" y="43.18" size="1.778" layer="95"/>
-<pinref part="GND2" gate="1" pin="GND"/>
-<wire x1="33.02" y1="43.18" x2="38.1" y2="43.18" width="0.1524" layer="91"/>
-<wire x1="38.1" y1="43.18" x2="38.1" y2="35.56" width="0.1524" layer="91"/>
+<wire x1="129.54" y1="111.76" x2="147.32" y2="111.76" width="0.1524" layer="91"/>
+<wire x1="147.32" y1="111.76" x2="167.64" y2="111.76" width="0.1524" layer="91"/>
+<wire x1="147.32" y1="111.76" x2="147.32" y2="104.14" width="0.1524" layer="91"/>
+<junction x="147.32" y="111.76"/>
+<pinref part="S2" gate="1" pin="P1"/>
+<wire x1="121.92" y1="111.76" x2="124.46" y2="111.76" width="0.1524" layer="91"/>
+<pinref part="S2" gate="1" pin="P"/>
+<wire x1="124.46" y1="111.76" x2="129.54" y2="111.76" width="0.1524" layer="91"/>
+<wire x1="121.92" y1="114.3" x2="124.46" y2="114.3" width="0.1524" layer="91"/>
+<wire x1="124.46" y1="114.3" x2="124.46" y2="111.76" width="0.1524" layer="91"/>
+<junction x="124.46" y="111.76"/>
+<pinref part="S1" gate="1" pin="S1"/>
+<wire x1="172.72" y1="111.76" x2="170.18" y2="111.76" width="0.1524" layer="91"/>
+<pinref part="S1" gate="1" pin="S"/>
+<wire x1="170.18" y1="111.76" x2="167.64" y2="111.76" width="0.1524" layer="91"/>
+<wire x1="172.72" y1="114.3" x2="170.18" y2="114.3" width="0.1524" layer="91"/>
+<wire x1="170.18" y1="114.3" x2="170.18" y2="111.76" width="0.1524" layer="91"/>
+<junction x="170.18" y="111.76"/>
+<pinref part="GND1" gate="1" pin="GND"/>
 </segment>
 </net>
@@
 </sheet>
 </sheets>
+<errors>
+</errors>
 </schematic>
 </drawing>
+<compatibility>
+<note version="8.2" severity="warning">
+Since Version 8.2, Eagle supports online libraries. The ids
+of those online libraries will not be understood (or retained)
+with this version.
+</note>
+</compatibility>
 </eagle>
