File: Hardware/ESP32-Final/esp32.brd (EAGLE design)
At the start: 27.5 x 71.2 mm, 53 parts, among them IC1 MCP73831/OT, Q2 SI2301, Q3 SI2301, Q4 SI2302, T1 BC847, T2 BC847, U1 ESP-WROOM-32, U2 AP2112K-3.3V

Commit message: Add files via upload
Parts:
- added R25: 47K, rcl:R0603
- C12: value 10uF -> 4.7uF
- C2, C3: value 10nF -> 4.7nF
- R1: value 10K -> 4K7
- R10: value 330K -> 220K
- R14, R18: value 10K -> 1K
Connections:
- removed net N$17: R24.1, U1.9
- net 3.3V: now also R24.1
- net GND: now also Q4.2, R25.1; no longer C11.1, Q4.3
- net N$15: now also C11.2
- net N$6: now also C11.1, Q4.3; no longer C11.2, Q4.2
- net VIN: now also R25.2
Routing:
- net N$17: track 53.1 -> 0.00 mm
- net N$6: track 19.3 -> 0.00 mm, vias 1 -> 0
- net N$1: track 8.05 -> 0.00 mm, vias 1 -> 0
- net GND: track 27.5 -> 24.2 mm, vias 16 -> 14
