File: Hardware/ESP32-Final/esp32.sch (EAGLE design)
At the start: 53 parts, among them IC1 MCP73831/OT, J1 1x6, Q2 SI2301, Q3 SI2301, Q4 SI2302, T1 BC847, T2 BC847, U1 ESP-WROOM-32, U2 AP2112K-3.3V

Commit message: Version 1.0.0
PCB v1.0.0
Parts:
- removed J1: 1x6, SparkFun-Connectors:6_PIN_SERIAL_TARGETSILK
- removed S2, S3: SMD-6.0X3.5MM, SparkFun-Switches:MOMENTARY-SWITCH-SPST-SMD-6.0X3.5MM
- added BTN1, BTN2: SPST.B3U-1000P(M), rinaldo:SPST.B3U-1000P(M)
- added U$1: 1X6, headers(2mm)(samtec):1X6
- renumbered LS1 to BZ1
Connections:
- removed net N$8: U$2.2
- net 3.3V: now also U$2.2
- net FLASH: now also BTN1.1; no longer S2.1
- net GND: now also BTN1.2, BTN2.1, U$1.1; no longer J1.GND, S2.2, S3.1
- net RESET: now also BTN2.2; no longer S3.2
- net RX: now also U$1.4; no longer J1.TXO
- net TX: now also U$1.5; no longer J1.RXI
Changed lines of the file:
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@@
 <part name="SUPPLY10" library="SparkFun-PowerSymbols" deviceset="3.3V" device=""/>
 <part name="GND22" library="SparkFun-PowerSymbols" deviceset="GND" device=""/>
-<part name="LS1" library="SparkFun-Electromechanical" deviceset="BUZZER" device="-PTH"/>
+<part name="BZ1" library="SparkFun-Electromechanical" deviceset="BUZZER" device="-PTH"/>
 <part name="GND26" library="SparkFun-PowerSymbols" deviceset="GND" device=""/>
 <part name="R20" library="resistor" library_urn="urn:adsk.eagle:library:348" deviceset="R-EU_" device="R0603" value="1K"/>
-<part name="J1" library="SparkFun-Connectors" deviceset="6_PIN_SERIAL_TARGET" device="SILK" value="1x6"/>
 <part name="GND4" library="SparkFun-PowerSymbols" deviceset="GND" device=""/>
 <part name="R17" library="resistor" library_urn="urn:adsk.eagle:library:348" deviceset="R-EU_" device="R0603" value="330R"/>
@@
 <part name="D1" library="SparkFun-DiscreteSemi" deviceset="DIODE-SCHOTTKY" device="-SS14" value="SS14"/>
 <part name="C9" library="rcl" library_urn="urn:adsk.eagle:library:334" deviceset="C-EU" device="C0603" value="10uF"/>
-<part name="S3" library="SparkFun-Switches" deviceset="MOMENTARY-SWITCH-SPST" device="-SMD-6.0X3.5MM" value="SMD-6.0X3.5MM"/>
-<part name="S2" library="SparkFun-Switches" deviceset="MOMENTARY-SWITCH-SPST" device="-SMD-6.0X3.5MM" value="SMD-6.0X3.5MM"/>
 <part name="R14" library="rcl" library_urn="urn:adsk.eagle:library:334" deviceset="R-EU_" device="R0603" value="10K"/>
 <part name="R18" library="rcl" library_urn="urn:adsk.eagle:library:334" deviceset="R-EU_" device="R0603" value="10K"/>
@@
 <part name="C3" library="rcl" library_urn="urn:adsk.eagle:library:334" deviceset="C-EU" device="C0603" value="10nF"/>
 <part name="C5" library="rcl" library_urn="urn:adsk.eagle:library:334" deviceset="C-EU" device="C0603" value="100nF"/>
+<part name="BTN1" library="rinaldo" deviceset="SPST" device=".B3U-1000P(M)" value=""/>
+<part name="BTN2" library="rinaldo" deviceset="SPST" device=".B3U-1000P(M)" value=""/>
+<part name="U$1" library="headers(2mm)(samtec)" deviceset="1X6" device=""/>
 </parts>
 <sheets>
 <sheet>
 <plain>
-<text x="15.24" y="162.56" size="1.778" layer="97">Reset</text>
-<text x="167.64" y="124.46" size="1.778" layer="97">BOOT</text>
+<text x="22.86" y="162.56" size="1.778" layer="97">Reset</text>
+<text x="160.02" y="127" size="1.778" layer="97">BOOT</text>
 <text x="-22.86" y="165.1" size="1.778" layer="97">FTDI</text>
 </plain>
@@
 <instance part="SUPPLY10" gate="G$1" x="152.4" y="134.62" rot="R270"/>
 <instance part="GND22" gate="1" x="149.86" y="139.7"/>
-<instance part="LS1" gate="G$1" x="218.44" y="157.48" smashed="yes" rot="R270">
+<instance part="BZ1" gate="G$1" x="218.44" y="157.48" smashed="yes" rot="R270">
 <attribute name="NAME" x="220.98" y="162.306" size="1.778" layer="95" font="vector"/>
 <attribute name="VALUE" x="221.234" y="147.32" size="1.778" layer="96" font="vector"/>
@@
 <instance part="GND26" gate="1" x="210.82" y="121.92"/>
 <instance part="R20" gate="G$1" x="193.04" y="144.78"/>
-<instance part="J1" gate="G$1" x="-15.24" y="149.86"/>
 <instance part="GND4" gate="1" x="0" y="157.48"/>
 <instance part="R17" gate="G$1" x="134.62" y="114.3"/>
@@
 </instance>
 <instance part="C9" gate="G$1" x="55.88" y="160.02"/>
-<instance part="S3" gate="G$1" x="25.4" y="157.48" smashed="yes">
-<attribute name="NAME" x="25.4" y="161.544" size="1.778" layer="95" font="vector" align="bottom-center"/>
-<attribute name="VALUE" x="27.94" y="156.972" size="1.778" layer="96" font="vector" align="top-center"/>
-</instance>
-<instance part="S2" gate="G$1" x="162.56" y="119.38" smashed="yes">
-<attribute name="NAME" x="162.56" y="123.444" size="1.778" layer="95" font="vector" align="bottom-center"/>
-<attribute name="VALUE" x="160.02" y="118.872" size="1.778" layer="96" font="vector" align="top-center"/>
-</instance>
 <instance part="R14" gate="G$1" x="-17.78" y="66.04" rot="R90"/>
 <instance part="R18" gate="G$1" x="-17.78" y="40.64" rot="R90"/>
@@
 <attribute name="VALUE" x="62.484" y="10.541" size="1.778" layer="96"/>
 </instance>
+<instance part="BTN1" gate="G$1" x="162.56" y="119.38"/>
+<instance part="BTN2" gate="G$1" x="25.4" y="157.48"/>
+<instance part="U$1" gate="G$1" x="-20.32" y="149.86"/>
 </instances>
 <busses>
@@
 <wire x1="172.72" y1="119.38" x2="172.72" y2="114.3" width="0.1524" layer="91"/>
 <pinref part="GND25" gate="1" pin="GND"/>
-<pinref part="S2" gate="G$1" pin="2"/>
 <wire x1="167.64" y1="119.38" x2="172.72" y2="119.38" width="0.1524" layer="91"/>
-</segment>
-<segment>
-<pinref part="U1" gate="G$1" pin="GND@4"/>
-<wire x1="121.92" y1="137.16" x2="142.24" y2="137.16" width="0.1524" layer="91"/>
+<pinref part="BTN1" gate="G$1" pin="2"/>
+<wire x1="165.1" y1="119.38" x2="167.64" y2="119.38" width="0.1524" layer="91"/>
+</segment>
+<segment>
 <wire x1="142.24" y1="137.16" x2="144.78" y2="137.16" width="0.1524" layer="91"/>
 <wire x1="144.78" y1="137.16" x2="144.78" y2="142.24" width="0.1524" layer="91"/>
@@
 <pinref part="GND22" gate="1" pin="GND"/>
 <wire x1="149.86" y1="144.78" x2="149.86" y2="142.24" width="0.1524" layer="91"/>
+<pinref part="U1" gate="G$1" pin="GND@4"/>
+<wire x1="121.92" y1="137.16" x2="142.24" y2="137.16" width="0.1524" layer="91"/>
 </segment>
 <segment>
@@
 </segment>
 <segment>
-<pinref part="J1" gate="G$1" pin="GND"/>
 <wire x1="-10.16" y1="157.48" x2="-7.62" y2="157.48" width="0.1524" layer="91"/>
 <wire x1="-7.62" y1="157.48" x2="-7.62" y2="162.56" width="0.1524" layer="91"/>
@@
 <wire x1="0" y1="162.56" x2="0" y2="160.02" width="0.1524" layer="91"/>
 <pinref part="GND4" gate="1" pin="GND"/>
+<wire x1="-17.78" y1="157.48" x2="-10.16" y2="157.48" width="0.1524" layer="91"/>
+<pinref part="U$1" gate="G$1" pin="1"/>
 </segment>
 <segment>
@@
 <wire x1="20.32" y1="157.48" x2="15.24" y2="157.48" width="0.1524" layer="91"/>
 <wire x1="15.24" y1="157.48" x2="15.24" y2="154.94" width="0.1524" layer="91"/>
-<pinref part="S3" gate="G$1" pin="1"/>
+<pinref part="BTN2" gate="G$1" pin="1"/>
+<wire x1="22.86" y1="157.48" x2="20.32" y2="157.48" width="0.1524" layer="91"/>
 </segment>
 <segment>
@@
 </segment>
 <segment>
-<wire x1="215.9" y1="104.14" x2="210.82" y2="104.14" width="0.1524" layer="91"/>
-<wire x1="210.82" y1="104.14" x2="210.82" y2="111.76" width="0.1524" layer="91"/>
-<pinref part="SUPPLY2" gate="G$1" pin="3.3V"/>
-<pinref part="U$2" gate="G$1" pin="1"/>
-</segment>
-<segment>
-<pinref part="SUPPLY8" gate="G$1" pin="3.3V"/>
-<wire x1="228.6" y1="111.76" x2="228.6" y2="109.22" width="0.1524" layer="91"/>
-</segment>
-<segment>
 <pinref part="C6" gate="G$1" pin="1"/>
 <wire x1="177.8" y1="66.04" x2="177.8" y2="71.12" width="0.1524" layer="91"/>
@@
 <junction x="177.8" y="73.66"/>
 </segment>
+<segment>
+<pinref part="U$2" gate="G$1" pin="1"/>
+<pinref part="SUPPLY2" gate="G$1" pin="3.3V"/>
+<wire x1="215.9" y1="104.14" x2="210.82" y2="104.14" width="0.1524" layer="91"/>
+<wire x1="210.82" y1="104.14" x2="210.82" y2="111.76" width="0.1524" layer="91"/>
+</segment>
+<segment>
+<pinref part="U$2" gate="G$1" pin="2"/>
+<pinref part="SUPPLY8" gate="G$1" pin="3.3V"/>
+<wire x1="223.52" y1="104.14" x2="228.6" y2="104.14" width="0.1524" layer="91"/>
+<wire x1="228.6" y1="104.14" x2="228.6" y2="111.76" width="0.1524" layer="91"/>
+</segment>
 </net>
 <net name="RESET" class="0">
@@
 <wire x1="35.56" y1="147.32" x2="40.64" y2="147.32" width="0.1524" layer="91"/>
 <junction x="40.64" y="147.32"/>
-<pinref part="S3" gate="G$1" pin="2"/>
 <wire x1="30.48" y1="157.48" x2="40.64" y2="157.48" width="0.1524" layer="91"/>
 <label x="55.88" y="147.32" size="1.778" layer="95"/>
+<pinref part="BTN2" gate="G$1" pin="2"/>
+<wire x1="30.48" y1="157.48" x2="27.94" y2="157.48" width="0.1524" layer="91"/>
 </segment>
 </net>
@@
 </segment>
 <segment>
-<pinref part="J1" gate="G$1" pin="RXI"/>
-<wire x1="-10.16" y1="147.32" x2="5.08" y2="147.32" width="0.1524" layer="91"/>
+<wire x1="-17.78" y1="147.32" x2="5.08" y2="147.32" width="0.1524" layer="91"/>
 <label x="0" y="147.32" size="1.778" layer="95"/>
+<pinref part="U$1" gate="G$1" pin="5"/>
 </segment>
 </net>
@@
 </segment>
 <segment>
-<pinref part="J1" gate="G$1" pin="TXO"/>
 <wire x1="-10.16" y1="149.86" x2="5.08" y2="149.86" width="0.1524" layer="91"/>
 <label x="0" y="149.86" size="1.778" layer="95"/>
+<wire x1="-17.78" y1="149.86" x2="-10.16" y2="149.86" width="0.1524" layer="91"/>
+<pinref part="U$1" gate="G$1" pin="4"/>
 </segment>
 </net>
@@
 <wire x1="147.32" y1="121.92" x2="147.32" y2="119.38" width="0.1524" layer="91"/>
 <junction x="147.32" y="119.38"/>
-<pinref part="S2" gate="G$1" pin="1"/>
 <label x="134.62" y="119.38" size="1.778" layer="95"/>
+<pinref part="BTN1" gate="G$1" pin="1"/>
+<wire x1="160.02" y1="119.38" x2="157.48" y2="119.38" width="0.1524" layer="91"/>
 </segment>
 </net>
@@
 <net name="N$3" class="0">
 <segment>
-<pinref part="LS1" gate="G$1" pin="2"/>
+<pinref part="BZ1" gate="G$1" pin="2"/>
 <wire x1="215.9" y1="154.94" x2="210.82" y2="154.94" width="0.1524" layer="91"/>
 <wire x1="210.82" y1="154.94" x2="210.82" y2="149.86" width="0.1524" layer="91"/>
@@
 <wire x1="215.9" y1="96.52" x2="205.74" y2="96.52" width="0.1524" layer="91"/>
 <label x="205.74" y="96.52" size="1.778" layer="95"/>
-</segment>
-</net>
-<net name="N$8" class="0">
-<segment>
-<wire x1="223.52" y1="104.14" x2="228.6" y2="104.14" width="0.1524" layer="91"/>
-<wire x1="228.6" y1="104.14" x2="228.6" y2="109.22" width="0.1524" layer="91"/>
-<pinref part="U$2" gate="G$1" pin="2"/>
 </segment>
 </net>
@@
 <net name="VIN" class="0">
 <segment>
-<pinref part="LS1" gate="G$1" pin="1"/>
+<pinref part="BZ1" gate="G$1" pin="1"/>
 <wire x1="215.9" y1="157.48" x2="210.82" y2="157.48" width="0.1524" layer="91"/>
 <wire x1="210.82" y1="157.48" x2="210.82" y2="162.56" width="0.1524" layer="91"/>

Commit message: Add files via upload
Parts:
- added R25: 47K, rcl:R-EU_R0603
- C12: value 10uF -> 4.7uF
- C2, C3: value 10nF -> 4.7nF
- R1: value 10K -> 4K7
- R10: value 330K -> 220K
- R14, R18: value 10K -> 1K
Connections:
- removed net N$17: R24.1, U1.IO33
- net 3.3V: now also R24.1
- net GND: now also Q4.S, R25.1; no longer C11.1, Q4.D
- net N$15: now also C11.2
- net N$6: now also C11.1, Q4.D; no longer C11.2, Q4.S
- net VIN: now also R25.2
Other:
- moved on the sheet: C11, C12, C13, C6, Q4, R10, R24, U2
